File: Hardware/SparkFun_Robo_HAT.sch (EAGLE design)
At the start: 139 parts, among them J1 RASPBERRYPI-40-PIN-GPIO_PTH_R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, J11 EXT MTR PWR, J18 ISP, J2 CORTEX_DEBUGPTH, J20 USB C, J7 EXT SERVO PWR, J8 EXT 5V PWR, Q1 310mA/60V/1.6Ω, Q23 20V/0.2A/8MHz/1.2Ω/1Vth, Q24 20V/0.2A/8MHz/1.2Ω/1Vth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

Commit message: Most labeling done, pwr and motor lines routed
Parts:
- removed C4: 0.1uF, SparkFun-Capacitors:0.1UF-0603-25V-(+80/-20%)
- removed LOGO3: OSHW-LOGOMINI, SparkFun-Aesthetics:OSHW-LOGOMINI
- removed LOGO5: SFE_LOGO_FLAME.1EXP, SparkFun-Aesthetics:SFE_LOGO_FLAME.1EXP
- removed TP22: TEST-POINT3X4, SparkFun-Connectors:TEST-POINT3X4
- added FRAME1: FRAME-LETTERNO_PACKAGE, SparkFun-Aesthetics:FRAME-LETTERNO_PACKAGE
- added J21, J22: (no value), SparkFun-Connectors:CONN_01PTH_NO_SILK_YES_STOP
- added TP9: TEST-POINT3X4, SparkFun-Connectors:TEST-POINT3X4
- FRAME3: value FRAME-LETTER -> FRAME-LEDGER; device SparkFun-Aesthetics:FRAME-LETTER -> SparkFun-Aesthetics:FRAME-LEDGER
Connections:
- net !RST renamed !ENC_RST
- net FSYNC_1.8V renamed !FSYNC_1.8V
- removed net !RESET: C23.1, J2.NRESET, TP13.1, U6G6.XRES
- removed net FSYNC_3.3V: Q27.D, R54.1
- removed net USB-5V: F2.2, JP2.2, Q10G$1.E, Q5.D, Q6G$1.E, Q7.D, Q8G$1.E, Q9.D
- new net !FSYNC_3.3V: J21.1, Q27.D, R54.1
- new net !MTR_RST: C23.1, J2.NRESET, J22.1, TP13.1, U6G6.XRES
- new net 5V: F2.2, J8.2, JP2.2, Q10G$1.E, Q5.D, Q6G$1.E, Q7.D, Q8G$1.E, Q9.D
- net !ENC_INT: now also J1.GP4
- net 3.3V: now also TP9.1; no longer TP22.1
- net GND: no longer C4.2
- net IMU_INT_3.3V: now also J1.CE1
- net PI-5V: no longer C4.1
- net VBUS: no longer J8.2
Other:
- note added: "*For frame synchronization support (3.3V Logic level)"
- note added: "Servo, Motor & Encoder Connections"
- note removed: "Motor & Encoder Connections"
- note removed: "Servo Connections"
- moved on the sheet: C10, C3, C5, C6, C7, C8, F2, J20, R10, R11

Commit message: Routing done, waiting on logo from marcom
Parts:
- removed TP10, TP13, TP14, TP15: TEST-POINTTP_15TH_THRU, SparkFun-Connectors:TEST-POINTTP_15TH_THRU
- removed TP16, TP17, TP9: TEST-POINT3X4, SparkFun-Connectors:TEST-POINT3X4
- removed TP4, TP6, TP7, TP8: TEST-POINT3, SparkFun-Connectors:TEST-POINT3
- TP11, TP12: value TEST-POINTTP_15TH_THRU -> TEST-POINT3X4; device SparkFun-Connectors:TEST-POINTTP_15TH_THRU -> SparkFun-Connectors:TEST-POINT3X4
- TP24: value TEST-POINT3X4 -> TEST-POINTTP_15TH_THRU; device SparkFun-Connectors:TEST-POINT3X4 -> SparkFun-Connectors:TEST-POINTTP_15TH_THRU
Connections:
- removed net AD0/SDO_VIN: JP15.2
- net !MTR_RST: no longer TP13.1
- net 3.3V: no longer TP10.1, TP7.1, TP9.1
- net 5V: now also C8.1, R1.2, R2.2, U1.VDD
- net AD0/SDO: now also JP15.2
- net GND: no longer TP17.1, TP8.1
- net P3.2: no longer TP4.1
- net P3.3: no longer TP6.1
- net PI-5V: no longer C8.1, R1.2, R2.2, U1.VDD
- net SCL_3.3V: no longer TP15.1
- net SDA_3.3V: no longer TP14.1
- net SERVO: no longer TP16.1
Other:
- note added: "ADR -> I2C Address ------------------- open -> 0x69 closed -> 0x68"
- note removed: "ADR -> I2C Address ------------------- open -> 0x69 closed -> 0x68 *Closing AD0 precludes SPI"
- note removed: "VIN 1.8V to 5.5V"
