File: Hardware/SparkFun_Robo_HAT.sch (EAGLE design)
At the start: 136 parts, among them J11 EXT MTR PWR, J18 ISP, J19 QWIIC_RIGHT_ANGLE, J2 RASPBERRYPI-40-PIN-GPIO_SMD_S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, J20 USB C, J23 CORTEX_JTAG_DEBUG_PTH, J7 EXT SERVO PWR, J8 EXT 5V PWR, Q1 310mA/60V/1.6Ω, Q23 20V/0.2A/8MHz/1.2Ω/1Vth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

Commit message: Added LOGO, improved GND pour flowing
-added LOGO to top and bottom silk
-rerouted some traces on right side of board near the EXT headers to allow for better GND flow
-added more gnd vias near SMD pads on stackable header package
-removed pesky test point values in SCH
Parts:
- J19: value QWIIC_RIGHT_ANGLE -> (none)
- J2: value RASPBERRYPI-40-PIN-GPIO_SMD_STACKABLE -> RASPBERRYPI-40-PIN-GPIO_SMD_STACKABLE_NOHOLES; device SparkFun-Connectors:RASPBERRYPI-40-PIN-GPIO_SMD_STACKABLE -> SparkFun-Connectors:RASPBERRYPI-40-PIN-GPIO_SMD_STACKABLE_NOHOLES
Changed lines of the file:
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@@
 <part name="LOGO1" library="SparkFun-Aesthetics" deviceset="SFE_LOGO_NAME_FLAME" device=".1_INCH"/>
 <part name="LOGO2" library="SparkFun-Aesthetics" deviceset="OSHW-LOGO" device="S" value="OSHW-LOGOS"/>
-<part name="J19" library="SparkFun-Connectors" deviceset="QWIIC_CONNECTOR" device="JS-1MM" value="QWIIC_RIGHT_ANGLE"/>
+<part name="J19" library="SparkFun-Connectors" deviceset="QWIIC_CONNECTOR" device="JS-1MM"/>
 <part name="GND1" library="SparkFun-PowerSymbols" deviceset="GND" device=""/>
 <part name="U$1" library="SparkFun-Aesthetics" deviceset="QWIIC_LOGO" device="_5MM" value="QWIIC_LOGO_5MM"/>
@@
 <part name="3.3V4" library="SparkFun-PowerSymbols" deviceset="VIN" device="" value="3.3V"/>
 <part name="3.3V5" library="SparkFun-PowerSymbols" deviceset="VIN" device="" value="3.3V"/>
-<part name="TP0" library="SparkFun-Connectors" deviceset="TEST-POINT" device="3X4" value="TEST-POINT3X4"/>
-<part name="TP1" library="SparkFun-Connectors" deviceset="TEST-POINT" device="3X4" value="TEST-POINT3X4"/>
-<part name="TP2" library="SparkFun-Connectors" deviceset="TEST-POINT" device="3X4" value="TEST-POINT3X4"/>
-<part name="TP3" library="SparkFun-Connectors" deviceset="TEST-POINT" device="3X4" value="TEST-POINT3X4"/>
-<part name="TP4" library="SparkFun-Connectors" deviceset="TEST-POINT" device="TP_15TH_THRU" value="TEST-POINTTP_15TH_THRU"/>
-<part name="TP5" library="SparkFun-Connectors" deviceset="TEST-POINT" device="TP_15TH_THRU" value="TEST-POINTTP_15TH_THRU"/>
+<part name="TP0" library="SparkFun-Connectors" deviceset="TEST-POINT" device="3X4" value=""/>
+<part name="TP1" library="SparkFun-Connectors" deviceset="TEST-POINT" device="3X4" value=""/>
+<part name="TP2" library="SparkFun-Connectors" deviceset="TEST-POINT" device="3X4" value=""/>
+<part name="TP3" library="SparkFun-Connectors" deviceset="TEST-POINT" device="3X4" value=""/>
+<part name="TP4" library="SparkFun-Connectors" deviceset="TEST-POINT" device="TP_15TH_THRU" value=""/>
+<part name="TP5" library="SparkFun-Connectors" deviceset="TEST-POINT" device="TP_15TH_THRU" value=""/>
 <part name="Q1" library="SparkFun-DiscreteSemi" deviceset="MOSFET-NCH" device="-2N7002PW" value="310mA/60V/1.6Ω"/>
 <part name="3.3V3" library="SparkFun-PowerSymbols" deviceset="VIN" device="" value="3.3V"/>
@@
 <part name="SUPPLY15" library="SparkFun-PowerSymbols" deviceset="VIN" device="" value="SERVO"/>
 <part name="5V5" library="SparkFun-PowerSymbols" deviceset="VIN" device="" value="PI-5V"/>
-<part name="TP6" library="SparkFun-Connectors" deviceset="TEST-POINT" device="3X4" value="TEST-POINT3X4"/>
+<part name="TP6" library="SparkFun-Connectors" deviceset="TEST-POINT" device="3X4" value=""/>
 <part name="5V2" library="SparkFun-PowerSymbols" deviceset="VIN" device="" value="PI-5V"/>
 <part name="C17" library="SparkFun-Capacitors" deviceset="1.0UF" device="-0402-16V-10%" value="1.0uF"/>
@@
 <part name="GND61" library="SparkFun-Aesthetics" deviceset="GND" device=""/>
 <part name="D2" library="SparkFun-LED" deviceset="LED-BLUE" device="0603" value="BLUE"/>
-<part name="TP7" library="SparkFun-Connectors" deviceset="TEST-POINT" device="3X4" value="TEST-POINT3X4"/>
-<part name="TP8" library="SparkFun-Connectors" deviceset="TEST-POINT" device="3X4" value="TEST-POINT3X4"/>
+<part name="TP7" library="SparkFun-Connectors" deviceset="TEST-POINT" device="3X4" value=""/>
+<part name="TP8" library="SparkFun-Connectors" deviceset="TEST-POINT" device="3X4" value=""/>
 <part name="U6" library="SparkFun-IC-Microcontroller" deviceset="PSOC4_4200_40QFN" device="" value="CY8C4245LQI-483"/>
-<part name="TP9" library="SparkFun-Connectors" deviceset="TEST-POINT" device="3" value="TEST-POINT3"/>
+<part name="TP9" library="SparkFun-Connectors" deviceset="TEST-POINT" device="3" value=""/>
 <part name="U7" library="SparkFun-Sensors" deviceset="ICM-20948" device="" value="9DoF IMU"/>
 <part name="C12" library="SparkFun-Capacitors" deviceset="0.1UF" device="-0603-25V-5%" value="0.1uF"/>
@@
 <part name="R3" library="SparkFun-Resistors" deviceset="5.1KOHM" device="5.1KOHM-0603-1/10W-1%" value="5.1k"/>
 <part name="R12" library="SparkFun-Resistors" deviceset="5.1KOHM" device="5.1KOHM-0603-1/10W-1%" value="5.1k"/>
-<part name="J2" library="SparkFun-Connectors" deviceset="RASPBERRYPI-40-PIN-GPIO" device="_SMD_STACKABLE" value="RASPBERRYPI-40-PIN-GPIO_SMD_STACKABLE"/>
+<part name="J2" library="SparkFun-Connectors" deviceset="RASPBERRYPI-40-PIN-GPIO" device="_SMD_STACKABLE_NOHOLES" value="RASPBERRYPI-40-PIN-GPIO_SMD_STACKABLE_NOHOLES"/>
 <part name="H9" library="SparkFun-Hardware" deviceset="STAND-OFF" device="TIGHT"/>
 <part name="H10" library="SparkFun-Hardware" deviceset="STAND-OFF" device="TIGHT"/>

Commit message: Design review changes
-added more GND stiching VIAs to middle area of board (MTR VIN trace kind of cutts top GND pour in half diagnoly)
-rotated IMU axis labels to read same as other silk
-separated imu axis labels on bottom silk
-removed GND traces from Cypress thermal pad to GND pads
-added more gnd vias under cypress
-removed TP15 name text in SCH
-changes SCH to 9V MAX EXT MTR input, *11v MAX with heat sink)
-added "default" text to IMU address paragraph
-added test points for IMU INT and DC motors lines and encoder lines
Parts:
- added TP10, TP11, TP12, TP13, TP14, TP15, TP16, TP17, TP18: TEST-POINT3X4, SparkFun-Connectors:TEST-POINT3X4
- TP9: value TEST-POINT3 -> TEST-POINT3X4; device SparkFun-Connectors:TEST-POINT3 -> SparkFun-Connectors:TEST-POINT3X4
Connections:
- net AOUT1: now also TP16.1
- net AOUT2: now also TP15.1
- net BOUT1: now also TP14.1
- net BOUT2: now also TP13.1
- net ENC1A_RAW: now also TP17.1
- net ENC1B_RAW: now also TP18.1
- net ENC2A_RAW: now also TP12.1
- net ENC2B_RAW: now also TP11.1
- net IMU_INT_3.3V: now also TP10.1
Other:
- note added: "11V MAX (with heat sink)"
- note added: "9V MAX"
- note added: "ADR -> I2C Address ------------------- open -> 0x69 (default) closed -> 0x68"
- note removed: "11V MAX"
- note removed: "ADR -> I2C Address ------------------- open -> 0x69 closed -> 0x68"
- moved on the sheet: TP0, TP1, TP2, TP3, TP4, TP5, TP6

Commit message: added test point to 3.3V rail
Parts:
- added TP19: TEST-POINTTP_15TH_THRU, SparkFun-Connectors:TEST-POINTTP_15TH_THRU
Connections:
- net 3.3V: now also TP19.1
Changed lines of the file:
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@@
 <part name="TP17" library="SparkFun-Connectors" deviceset="TEST-POINT" device="3X4" value=""/>
 <part name="TP18" library="SparkFun-Connectors" deviceset="TEST-POINT" device="3X4" value=""/>
+<part name="3.3V9" library="SparkFun-PowerSymbols" deviceset="VIN" device="" value="3.3V"/>
+<part name="TP19" library="SparkFun-Connectors" deviceset="TEST-POINT" device="TP_15TH_THRU" value=""/>
 </parts>
 <sheets>
@@
 <attribute name="VALUE" x="200.66" y="106.68" size="1.778" layer="96" font="vector"/>
 </instance>
+<instance part="3.3V9" gate="G$1" x="200.66" y="132.08" smashed="yes" rot="MR0">
+<attribute name="VALUE" x="200.66" y="134.874" size="1.778" layer="96" font="vector" rot="MR0" align="bottom-center"/>
+</instance>
+<instance part="TP19" gate="G$1" x="203.2" y="129.54" smashed="yes">
+<attribute name="NAME" x="206.756" y="128.778" size="1.778" layer="95" font="vector"/>
+<attribute name="VALUE" x="200.66" y="127" size="1.778" layer="96" font="vector"/>
+</instance>
 </instances>
 <busses>
@@
 <junction x="88.9" y="73.66"/>
 </segment>
-</net>
+<segment>
+<pinref part="3.3V9" gate="G$1" pin="VIN"/>
+<pinref part="TP19" gate="G$1" pin="1"/>
+<wire x1="203.2" y1="129.54" x2="200.66" y2="129.54" width="0.1524" layer="91"/>
+<wire x1="200.66" y1="129.54" x2="200.66" y2="132.08" width="0.1524" layer="91"/>
+</segment>
+</net>

Commit message: fixed vector font issue on servo "~"
-bumped version to v11
-also updated the "+" and "-" symbols on servo headers and encoder terminals (on both top silk and bottom silk) I drew everything with wires so they look clean and will hold position through the panelizer ulp tool
Other:
- note added: "v11"
- note removed: "v10"
Changed lines of the file:
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@@
 <grid distance="0.1" unitdist="inch" unit="inch" style="lines" multiple="1" display="no" altdistance="0.01" altunitdist="inch" altunit="inch"/>
 <layers>
-<layer number="1" name="Top" color="4" fill="1" visible="yes" active="no"/>
-<layer number="2" name="Route2" color="1" fill="3" visible="yes" active="no"/>
-<layer number="3" name="Route3" color="4" fill="3" visible="yes" active="no"/>
-<layer number="4" name="Route4" color="1" fill="4" visible="yes" active="no"/>
-<layer number="5" name="Route5" color="4" fill="4" visible="yes" active="no"/>
-<layer number="6" name="Route6" color="1" fill="8" visible="yes" active="no"/>
-<layer number="7" name="Route7" color="4" fill="8" visible="yes" active="no"/>
-<layer number="8" name="Route8" color="1" fill="2" visible="yes" active="no"/>
-<layer number="9" name="Route9" color="4" fill="2" visible="yes" active="no"/>
-<layer number="10" name="Route10" color="1" fill="7" visible="yes" active="no"/>
-<layer number="11" name="Route11" color="4" fill="7" visible="yes" active="no"/>
-<layer number="12" name="Route12" color="1" fill="5" visible="yes" active="no"/>
-<layer number="13" name="Route13" color="4" fill="5" visible="yes" active="no"/>
-<layer number="14" name="Route14" color="1" fill="6" visible="yes" active="no"/>
-<layer number="15" name="Route15" color="4" fill="6" visible="yes" active="no"/>
-<layer number="16" name="Bottom" color="1" fill="1" visible="yes" active="no"/>
-<layer number="17" name="Pads" color="2" fill="1" visible="yes" active="no"/>
-<layer number="18" name="Vias" color="2" fill="1" visible="yes" active="no"/>
-<layer number="19" name="Unrouted" color="6" fill="1" visible="yes" active="no"/>
-<layer number="20" name="Dimension" color="24" fill="1" visible="yes" active="no"/>
-<layer number="21" name="tPlace" color="16" fill="1" visible="yes" active="no"/>
-<layer number="22" name="bPlace" color="14" fill="1" visible="yes" active="no"/>
-<layer number="23" name="tOrigins" color="15" fill="1" visible="yes" active="no"/>
-<layer number="24" name="bOrigins" color="15" fill="1" visible="yes" active="no"/>
-<layer number="25" name="tNames" color="7" fill="1" visible="yes" active="no"/>
-<layer number="26" name="bNames" color="7" fill="1" visible="yes" active="no"/>
-<layer number="27" name="tValues" color="7" fill="1" visible="yes" active="no"/>
-<layer number="28" name="bValues" color="7" fill="1" visible="yes" active="no"/>
+<layer number="1" name="Top" color="4" fill="1" visible="no" active="no"/>
+<layer number="2" name="Route2" color="1" fill="3" visible="no" active="no"/>
+<layer number="3" name="Route3" color="4" fill="3" visible="no" active="no"/>
+<layer number="4" name="Route4" color="1" fill="4" visible="no" active="no"/>
+<layer number="5" name="Route5" color="4" fill="4" visible="no" active="no"/>
+<layer number="6" name="Route6" color="1" fill="8" visible="no" active="no"/>
+<layer number="7" name="Route7" color="4" fill="8" visible="no" active="no"/>
+<layer number="8" name="Route8" color="1" fill="2" visible="no" active="no"/>
+<layer number="9" name="Route9" color="4" fill="2" visible="no" active="no"/>
+<layer number="10" name="Route10" color="1" fill="7" visible="no" active="no"/>
+<layer number="11" name="Route11" color="4" fill="7" visible="no" active="no"/>
+<layer number="12" name="Route12" color="1" fill="5" visible="no" active="no"/>
+<layer number="13" name="Route13" color="4" fill="5" visible="no" active="no"/>
+<layer number="14" name="Route14" color="1" fill="6" visible="no" active="no"/>
+<layer number="15" name="Route15" color="4" fill="6" visible="no" active="no"/>
+<layer number="16" name="Bottom" color="1" fill="1" visible="no" active="no"/>
+<layer number="17" name="Pads" color="2" fill="1" visible="no" active="no"/>
+<layer number="18" name="Vias" color="2" fill="1" visible="no" active="no"/>
+<layer number="19" name="Unrouted" color="6" fill="1" visible="no" active="no"/>
+<layer number="20" name="Dimension" color="24" fill="1" visible="no" active="no"/>
+<layer number="21" name="tPlace" color="16" fill="1" visible="no" active="no"/>
+<layer number="22" name="bPlace" color="14" fill="1" visible="no" active="no"/>
+<layer number="23" name="tOrigins" color="15" fill="1" visible="no" active="no"/>
+<layer number="24" name="bOrigins" color="15" fill="1" visible="no" active="no"/>
+<layer number="25" name="tNames" color="7" fill="1" visible="no" active="no"/>
+<layer number="26" name="bNames" color="7" fill="1" visible="no" active="no"/>
+<layer number="27" name="tValues" color="7" fill="1" visible="no" active="no"/>
+<layer number="28" name="bValues" color="7" fill="1" visible="no" active="no"/>
 <layer number="29" name="tStop" color="7" fill="3" visible="no" active="no"/>
 <layer number="30" name="bStop" color="7" fill="6" visible="no" active="no"/>
@@
 <layer number="35" name="tGlue" color="7" fill="4" visible="no" active="no"/>
 <layer number="36" name="bGlue" color="7" fill="5" visible="no" active="no"/>
-<layer number="37" name="tTest" color="7" fill="1" visible="yes" active="no"/>
-<layer number="38" name="bTest" color="7" fill="1" visible="yes" active="no"/>
+<layer number="37" name="tTest" color="7" fill="1" visible="no" active="no"/>
+<layer number="38" name="bTest" color="7" fill="1" visible="no" active="no"/>
 <layer number="39" name="tKeepout" color="4" fill="11" visible="no" active="no"/>
 <layer number="40" name="bKeepout" color="1" fill="11" visible="no" active="no"/>
@@
 <layer number="44" name="Drills" color="7" fill="1" visible="no" active="no"/>
 <layer number="45" name="Holes" color="7" fill="1" visible="no" active="no"/>
-<layer number="46" name="Milling" color="3" fill="1" visible="yes" active="no"/>
-<layer number="47" name="Measures" color="7" fill="1" visible="yes" active="no"/>
-<layer number="48" name="Document" color="13" fill="7" visible="yes" active="no"/>
-<layer number="49" name="Reference" color="13" fill="1" visible="yes" active="no"/>
-<layer number="50" name="dxf" color="7" fill="1" visible="yes" active="no"/>
-<layer number="51" name="tDocu" color="6" fill="1" visible="yes" active="no"/>
-<layer number="52" name="bDocu" color="7" fill="1" visible="yes" active="no"/>
-<layer number="53" name="tGND_GNDA" color="7" fill="9" visible="yes" active="no"/>
-<layer number="54" name="bGND_GNDA" color="1" fill="9" visible="yes" active="no"/>
-<layer number="56" name="wert" color="7" fill="1" visible="yes" active="no"/>
-<layer number="57" name="tCAD" color="7" fill="1" visible="yes" active="no"/>
-<layer number="59" name="tCarbon" color="7" fill="1" visible="yes" active="no"/>
-<layer number="60" name="bCarbon" color="7" fill="1" visible="yes" active="no"/>
+<layer number="46" name="Milling" color="3" fill="1" visible="no" active="no"/>
+<layer number="47" name="Measures" color="7" fill="1" visible="no" active="no"/>
+<layer number="48" name="Document" color="13" fill="7" visible="no" active="no"/>
+<layer number="49" name="Reference" color="13" fill="1" visible="no" active="no"/>
+<layer number="50" name="dxf" color="7" fill="1" visible="no" active="no"/>
+<layer number="51" name="tDocu" color="6" fill="1" visible="no" active="no"/>
+<layer number="52" name="bDocu" color="7" fill="1" visible="no" active="no"/>
+<layer number="53" name="tGND_GNDA" color="7" fill="9" visible="no" active="no"/>
+<layer number="54" name="bGND_GNDA" color="1" fill="9" visible="no" active="no"/>
+<layer number="56" name="wert" color="7" fill="1" visible="no" active="no"/>
+<layer number="57" name="tCAD" color="7" fill="1" visible="no" active="no"/>
+<layer number="59" name="tCarbon" color="7" fill="1" visible="no" active="no"/>
+<layer number="60" name="bCarbon" color="7" fill="1" visible="no" active="no"/>
 <layer number="88" name="SimResults" color="9" fill="1" visible="no" active="yes"/>
 <layer number="89" name="SimProbes" color="9" fill="1" visible="no" active="yes"/>
@@
 <plain>
 <text x="349.758" y="11.43" size="2.54" layer="94" font="vector">Pete Lewis</text>
-<text x="421.64" y="6.604" size="2.54" layer="94" font="vector" ratio="12">v10</text>
+<text x="421.64" y="6.604" size="2.54" layer="94" font="vector" ratio="12">v11</text>
 <wire x1="139.7" y1="152.4" x2="139.7" y2="91.44" width="0.3048" layer="97" style="longdash"/>
 <wire x1="139.7" y1="91.44" x2="139.7" y2="0" width="0.3048" layer="97" style="longdash"/>
@@
 <text x="166.624" y="11.43" size="2.54" layer="94" font="vector">Pete Lewis</text>
 <text x="5.08" y="177.8" size="3.81" layer="94" font="vector">Motor Driver IC - PSoC I/O</text>
-<text x="237.49" y="7.62" size="2.54" layer="94" font="vector">v10</text>
+<text x="237.49" y="7.62" size="2.54" layer="94" font="vector">v11</text>
 <text x="123.698" y="18.288" size="1.27" layer="97" font="vector" rot="MR180">P3.2 swd_io[0]
 P3.3 swd_clk[0]
@@
 <text x="261.874" y="11.176" size="1.778" layer="97" font="vector">*For frame synchronization support
 (3.3V Logic level)</text>
-<text x="421.386" y="7.366" size="2.54" layer="94" font="vector">v10</text>
+<text x="421.386" y="7.366" size="2.54" layer="94" font="vector">v11</text>
 <text x="349.758" y="11.43" size="2.54" layer="94" font="vector">Pete Lewis</text>
 </plain>
