File: Hardware/SparkFun_Auto_pHAT.brd (EAGLE design)
At the start: 65.1 x 57 mm, 235 parts, among them J11 EXT MTR PWR, J18 ISP, J2 RASPBERRYPI-40-PIN-GPIO_SMD_S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, J20 USB C, J23 CORTEX_JTAG_DEBUG_PTH, J7 EXT SERVO PWR, J8 EXT 5V PWR, Q1 310mA/60V/1.6Ω, Q23 20V/0.2A/8MHz/1.2Ω/1Vth, Q24 20V/0.2A/8MHz/1.2Ω/1Vth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

Commit message: Added Address jumpers for Servo IC
-Added 3 address jumpers to Servo IC. (includes a BOM change to include 3 more 10K resistors) This will allow for up to 8 different addresses. Note, A4 and A5 are permenantly connected to GND.
-Added address table to SCH for address jumpers.
-increased one of the "fan" holes to allow for even more airflow using the SHIM fan.
Parts:
- added JP1, JP5, JP6: JUMPER-PAD-2, SparkFun-Jumpers:SMT-JUMPER_2_NC_TRACE_NO-SILK
- added R17, R18, R19: 10k, SparkFun-Resistors:0603@1
- added U$28: (no value), buzzard_labels (2):SRV_ADD0
- added U$41: (no value), buzzard_labels:05
- added U$42: (no value), buzzard_labels:16
- added U$45: (no value), buzzard_labels:27
- added U$46: (no value), buzzard_labels (3):MTR0
- moved LOGO1 40.0 mm to (6.38, 12.3)
- moved U$83 11.0 mm to (39.5, 43.0)
- moved LOGO4 3.05 mm to (11.1, 36.4)
- moved JP13 3.05 mm to (14.7, 35.6)
- moved U$49 3.02 mm to (14.2, 35.6)
- moved JP15 0.71 mm to (31.6, 37.5)
- moved U$39 0.66 mm to (31.1, 37.5)
Connections:
- new net ADD_A0: JP1.2, R18.1, U1.1
- new net ADD_A1: JP5.2, R17.1, U1.2
- new net ADD_A2: JP6.2, R19.1, U1.3
- net 5V: now also R17.2, R18.2, R19.2
- net GND: now also JP1.1, JP5.1, JP6.1, U1.4, U1.5
Routing:
- net ADD_A2: track 0.00 -> 8.51 mm, vias 0 -> 1
- net 5V: track 106.2 -> 113.7 mm, vias 5 -> 6
- net ADD_A1: track 0.00 -> 6.71 mm, vias 0 -> 1
- net ADD_A0: track 0.00 -> 6.68 mm, vias 0 -> 1
- net !MTR_RST: track 54.4 -> 51.6 mm
- net !ENC_RST: track 88.9 -> 91.6 mm
- net 3.3V: track 322.5 -> 321.3 mm
- net AD0/SDO: track 13.7 -> 14.4 mm

Commit message: Changed SVR ADD label to SVR ADR (to match others)
Parts:
- removed U$28: (no value), buzzard_labels (2):SRV_ADD0
- added U$47: (no value), buzzard_labels (4):SRV_ADR0
Changed lines of the file:
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@@
 <hole x="34.7218" y="28.5242" drill="1"/>
 <hole x="29.6164" y="35.6362" drill="1"/>
-<wire x1="50.899059375" y1="26.055321875" x2="43.957240625" y2="26.042621875" width="0.2032" layer="22"/>
-<wire x1="50.89651875" y1="31.478221875" x2="50.899059375" y2="26.055321875" width="0.2032" layer="22"/>
-<wire x1="43.96231875" y1="31.478221875" x2="43.964859375" y2="26.055321875" width="0.2032" layer="22"/>
+<wire x1="50.619659375" y1="26.055321875" x2="44.262040625" y2="26.042621875" width="0.2032" layer="22"/>
+<wire x1="50.64251875" y1="32.062421875" x2="50.619659375" y2="26.055321875" width="0.2032" layer="22"/>
+<wire x1="44.29251875" y1="32.062421875" x2="44.269659375" y2="26.055321875" width="0.2032" layer="22"/>
 <rectangle x1="46.482" y1="24.0538" x2="46.5328" y2="24.3586" layer="41"/>
 <hole x="19.1516" y="37.3888" drill="3.048"/>
@@
 <attribute name="VALUE" x="45.7454" y="21.7678" size="0.6096" layer="27" font="vector" ratio="20" rot="R270" align="top-center"/>
 </element>
-<element name="U$28" library="buzzard_labels (2)" package="SRV_ADD0" value="" x="51.4858" y="31.3436" smashed="yes" rot="MR0"/>
 <element name="U$41" library="buzzard_labels" package="05" value="" x="46.962059375" y="29.50718125" smashed="yes" rot="MR0"/>
 <element name="U$42" library="buzzard_labels" package="16" value="" x="48.981359375" y="29.474159375" smashed="yes" rot="MR0"/>
 <element name="U$45" library="buzzard_labels" package="27" value="" x="50.784759375" y="29.4513" smashed="yes" rot="MR0"/>
 <element name="U$46" library="buzzard_labels (3)" package="MTR0" value="" x="4.2418" y="14.605" smashed="yes" rot="R270"/>
+<element name="U$47" library="buzzard_labels (4)" package="SRV_ADR0" value="" x="51.4858" y="31.3436" smashed="yes" rot="MR0"/>
 </elements>
 <signals>
