File: Hardware/Production/SparkFun_Auto_pHAT-Panel.brd (EAGLE design)
At the start: 226.4 x 136.6 mm, 1404 parts, among them J100 ISP, J105 EXT SERVO PWR, J106 EXT 5V PWR, J109 CORTEX_JTAG_DEBUG_PTH, J11 EXT MTR PWR, J110 RASPBERRYPI-40-PIN-GPIO_SMD_S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, J112 USB C, J113 EXT MTR PWR, J122 ISP, J127 EXT SERVO PWR, J128 EXT 5V PWR, J131 CORTEX_JTAG_DEBUG_PTH, J132 RASPBERRYPI-40-PIN-GPIO_SMD_S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, J18 ISP, J2 RASPBERRYPI-40-PIN-GPIO_SMD_S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, J20 USB C, J23 CORTEX_JTAG_DEBUG_PTH, J24 USB C, J25 EXT MTR PWR, J34 ISP, J39 EXT SERVO PWR, J40 EXT 5V PWR, J43 CORTEX_JTAG_DEBUG_PTH, J44 RASPBERRYPI-40-PIN-GPIO_SMD_S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, J46 USB C, J47 EXT MTR PWR, J56 ISP, J61 EXT SERVO PWR, J62 EXT 5V PWR, J65 CORTEX_JTAG_DEBUG_PTH, J66 RASPBERRYPI-40-PIN-GPIO_SMD_S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, J68 USB C, J69 EXT MTR PWR, J7 EXT SERVO PWR, J78 ISP, J8 EXT 5V PWR, J83 EXT SERVO PWR, J84 EXT 5V PWR, J87 CORTEX_JTAG_DEBUG_PTH, J88 RASPBERRYPI-40-PIN-GPIO_SMD_S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, J90 USB C, J91 EXT MTR PWR, Q1 310mA/60V/1.6Ω, Q11 20V/4.2A/52mΩ/1.4W, Q13 20V/4.2A/52mΩ/1.4W, Q15 20V/4.2A/52mΩ/1.4W, Q17 20V/0.2A/8MHz/1.2Ω/1Vth, Q18 20V/0.2A/8MHz/1.2Ω/1Vth, Q19 20V/0.2A/8MHz/1.2Ω/1Vth, Q2 310mA/60V/1.6Ω, Q20 20V/0.2A/8MHz/1.2Ω/1Vth, Q21 310mA/60V/1.6Ω, Q22 310mA/60V/1.6Ω, Q23 20V/0.2A/8MHz/1.2Ω/1Vth, Q24 20V/0.2A/8MHz/1.2Ω/1Vth, Q25 20V/4.2A/52mΩ/1.4W, Q27 20V/0.2A/8MHz/1.2Ω/1Vth, Q28 20V/0.2A/8MHz/1.2Ω/1Vth, Q29 20V/4.2A/52mΩ/1.4W, Q3 310mA/60V/1.6Ω, Q31 20V/4.2A/52mΩ/1.4W, Q33 20V/0.2A/8MHz/1.2Ω/1Vth, Q34 20V/0.2A/8MHz/1.2Ω/1Vth, Q35 20V/0.2A/8MHz/1.2Ω/1Vth, Q36 20V/0.2A/8MHz/1.2Ω/1Vth, Q37 310mA/60V/1.6Ω, Q38 310mA/60V/1.6Ω, Q39 20V/4.2A/52mΩ/1.4W, Q4 310mA/60V/1.6Ω, Q41 20V/4.2A/52mΩ/1.4W, Q43 20V/4.2A/52mΩ/1.4W, Q45 20V/0.2A/8MHz/1.2Ω/1Vth, Q46 20V/0.2A/8MHz/1.2Ω/1Vth, Q47 20V/0.2A/8MHz/1.2Ω/1Vth, Q48 20V/0.2A/8MHz/1.2Ω/1Vth, Q49 310mA/60V/1.6Ω, Q5 20V/4.2A/52mΩ/1.4W, Q50 310mA/60V/1.6Ω, Q51 20V/4.2A/52mΩ/1.4W, Q53 20V/4.2A/52mΩ/1.4W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

Commit message: v12 gerbers
Parts:
- added JP55, JP65, JP66, JP67: JUMPER-PAD-2, SparkFun-Jumpers:SMT-JUMPER_2_NO_NO-SILK
- added JP56, JP57, JP68, JP69: ADR, SparkFun-Jumpers:SMT-JUMPER_2_NO_SILK
- added JP58, JP59, JP60, JP64, JP70, JP71, JP72: JUMPER-PAD-2, SparkFun-Jumpers:SMT-JUMPER_2_NC_TRACE_NO-SILK
- added JP61: FUSE BP, SparkFun-Jumpers:SMT-JUMPER_2_NO_SILK
- added JP62: I2C, SparkFun-Jumpers:SMT-JUMPER_3_2-NC_TRACE_SILK
- added JP63: PI ISO, SparkFun-Jumpers:SMT-JUMPER_2_NC_TRACE_SILK
- added R211, R225: 2.2k, SparkFun-Resistors:0402-TIGHT
- added R212, R213, R214, R215, R216, R217, R218, R219, R220, R221, R226, R227, R228: 10k, SparkFun-Resistors:0603@1
- added R222, R223, R224: 5.1k, SparkFun-Resistors:0603@1
- added U$529, U$558: (no value), buzzard_labels (5):33
- added U$530: (no value), buzzard_labels (6):ENC_INT12
- added U$531: (no value), buzzard_labels (6):ENC_ADR11
- added U$532: (no value), buzzard_labels (6):FUSE_BP10
- added U$533: (no value), buzzard_labels (6):IMU_ADR9
- added U$534: (no value), buzzard_labels (7):MTR_ADR0
- added U$535: (no value), buzzard_labels (1):EXT_PWR_INPUTS3
- added U$536: (no value), buzzard_labels (6):5V3
- added U$537: (no value), buzzard_labels (6):#ENC_RST6
- added U$538: (no value), buzzard_labels (6):#MTR_RST7
- added U$539: (no value), buzzard_labels (6):#FSYNC8
- added U$540, U$541, U$542: (no value), buzzard_labels:GND3
- added U$543: (no value), buzzard_labels (8):#ENC_INT0
- added U$544, U$545: (no value), buzzard_labels (2):B15
- added U$546: (no value), buzzard_labels (2):ENC112
- added U$547: (no value), buzzard_labels (2):ENC213
- added U$548, U$549: (no value), buzzard_labels (2):A14
- added U$550: (no value), buzzard_labels (3):MTRA0
- added U$551: (no value), buzzard_labels (3):MTRB1
- added U$552, U$553: (no value), buzzard_labels (4):10
- added U$554, U$555: (no value), buzzard_labels (4):21
- added U$556: (no value), buzzard_labels (5):00
- added U$557: (no value), buzzard_labels (5):22
- added U$559: (no value), buzzard_labels (5):11
- added U$560, U$561: (no value), robohat:AUTOHAT-LOGO
- added U$562, U$563: (no value), autophat:1X06_2.54_SCREWTERM_PIN_REF
- added U$564: (no value), buzzard_labels:SRV_5#6V1
- added U$565: (no value), buzzard_labels (1):MTR_5#9V0
- added U$566: (no value), buzzard_labels:05
- added U$567: (no value), buzzard_labels:16
- added U$568: (no value), buzzard_labels:27
- added U$569: (no value), buzzard_labels (3):MTR0
- added U$570: (no value), buzzard_labels (4):SRV_ADR0
- J114, J116, J117, J119, J13, J14, J16, J26, J28, J29, J31, J48, J50, J51, J53, J70, J72, J73, J75, J9, J92, J94, J95, J97: device SparkFun-Connectors:1X02_2.54_SCREWTERM -> autophat:1X02_2.54_SCREWTERM_LG_DRILL
- JP1, JP28, JP46: value FUSE BP -> JUMPER-PAD-2; device SparkFun-Jumpers:SMT-JUMPER_2_NO_SILK -> SparkFun-Jumpers:SMT-JUMPER_2_NC_TRACE_NO-SILK
- JP14, JP51: value JUMPER-PAD-2 -> PI ISO; device SparkFun-Jumpers:SMT-JUMPER_2_NO_NO-SILK -> SparkFun-Jumpers:SMT-JUMPER_2_NC_TRACE_SILK
- JP16, JP23, JP24, JP34, JP52: device SparkFun-Jumpers:SMT-JUMPER_2_NO_NO-SILK -> SparkFun-Jumpers:SMT-JUMPER_2_NC_TRACE_NO-SILK
- JP17, JP18, JP53, JP54: value ADR -> JUMPER-PAD-2; device SparkFun-Jumpers:SMT-JUMPER_2_NO_SILK -> SparkFun-Jumpers:SMT-JUMPER_2_NO_NO-SILK
- JP19: value FUSE BP -> JUMPER-PAD-2; device SparkFun-Jumpers:SMT-JUMPER_2_NO_SILK -> SparkFun-Jumpers:SMT-JUMPER_2_NO_NO-SILK
- JP20: value I2C -> ADR; device SparkFun-Jumpers:SMT-JUMPER_3_2-NC_TRACE_SILK -> SparkFun-Jumpers:SMT-JUMPER_2_NO_SILK
- JP21: value PI ISO -> ADR; device SparkFun-Jumpers:SMT-JUMPER_2_NC_TRACE_SILK -> SparkFun-Jumpers:SMT-JUMPER_2_NO_SILK
- JP25: value JUMPER-PAD-2 -> FUSE BP; device SparkFun-Jumpers:SMT-JUMPER_2_NO_NO-SILK -> SparkFun-Jumpers:SMT-JUMPER_2_NO_SILK
- JP26: value ADR -> I2C; device SparkFun-Jumpers:SMT-JUMPER_2_NO_SILK -> SparkFun-Jumpers:SMT-JUMPER_3_2-NC_TRACE_SILK
- JP27: value ADR -> PI ISO; device SparkFun-Jumpers:SMT-JUMPER_2_NO_SILK -> SparkFun-Jumpers:SMT-JUMPER_2_NC_TRACE_SILK
- JP29: value I2C -> JUMPER-PAD-2; device SparkFun-Jumpers:SMT-JUMPER_3_2-NC_TRACE_SILK -> SparkFun-Jumpers:SMT-JUMPER_2_NO_NO-SILK
- JP30: value PI ISO -> JUMPER-PAD-2; device SparkFun-Jumpers:SMT-JUMPER_2_NC_TRACE_SILK -> SparkFun-Jumpers:SMT-JUMPER_2_NO_NO-SILK
- JP31: device SparkFun-Jumpers:SMT-JUMPER_2_NC_TRACE_NO-SILK -> SparkFun-Jumpers:SMT-JUMPER_2_NO_NO-SILK
- JP32, JP33: value JUMPER-PAD-2 -> ADR; device SparkFun-Jumpers:SMT-JUMPER_2_NO_NO-SILK -> SparkFun-Jumpers:SMT-JUMPER_2_NO_SILK
- JP35, JP36: value ADR -> JUMPER-PAD-2; device SparkFun-Jumpers:SMT-JUMPER_2_NO_SILK -> SparkFun-Jumpers:SMT-JUMPER_2_NC_TRACE_NO-SILK
- JP47, JP5: value I2C -> JUMPER-PAD-2; device SparkFun-Jumpers:SMT-JUMPER_3_2-NC_TRACE_SILK -> SparkFun-Jumpers:SMT-JUMPER_2_NC_TRACE_NO-SILK
- JP48, JP6: value PI ISO -> JUMPER-PAD-2; device SparkFun-Jumpers:SMT-JUMPER_2_NC_TRACE_SILK -> SparkFun-Jumpers:SMT-JUMPER_2_NC_TRACE_NO-SILK
- JP49, JP7: value JUMPER-PAD-2 -> FUSE BP; device SparkFun-Jumpers:SMT-JUMPER_2_NC_TRACE_NO-SILK -> SparkFun-Jumpers:SMT-JUMPER_2_NO_SILK
- JP50, JP8: value JUMPER-PAD-2 -> I2C; device SparkFun-Jumpers:SMT-JUMPER_2_NO_NO-SILK -> SparkFun-Jumpers:SMT-JUMPER_3_2-NC_TRACE_SILK
- R102, R103, R104, R137, R138, R139, R145, R174, R180, R181, R21, R23, R67, R68, R69, R75, R76: value 5.1k -> 10k
- R105, R122, R124, R126, R140, R156, R160, R175, R191, R192, R193, R194, R86, R88: value 2.2k -> 10k; device SparkFun-Resistors:0402-TIGHT -> SparkFun-Resistors:0603@1
- R108, R109, R148, R185, R28, R71, R72, R82: value 10k -> 5.1k
- R111, R172, R173, R207, R208, R209: value 5.1k -> 2.2k; device SparkFun-Resistors:0603@1 -> SparkFun-Resistors:0402-TIGHT
- R112, R114, R116, R151, R182, R24, R31, R77, R79: value 47k -> 10k
- R118, R153, R154, R188, R189, R34, R84: value 1 -> 10k
- R119: value 1 -> 5.1k
- R120: value 470 -> 5.1k
- R121, R123, R125, R159, R161, R87: value 2.2k -> 47k; device SparkFun-Resistors:0402-TIGHT -> SparkFun-Resistors:0603@1
- R127, R128, R165, R166, R203, R204: value 10k -> 1
- R129, R167, R205: value 10k -> 470
- R130, R131, R132, R133, R134, R135, R168, R169, R170, R171, R187, R206, R57, R58, R59, R73, R92, R93, R94, R95, R96, R97: value 10k -> 2.2k; device SparkFun-Resistors:0603@1 -> SparkFun-Resistors:0402-TIGHT
- R147, R184, R186, R29, R81: value 47k -> 5.1k
- R149: value 47k -> 2.2k; device SparkFun-Resistors:0603@1 -> SparkFun-Resistors:0402-TIGHT
- R155, R190, R36: value 470 -> 10k
- R157, R158, R195, R196, R70: value 2.2k -> 5.1k; device SparkFun-Resistors:0402-TIGHT -> SparkFun-Resistors:0603@1
- R163, R197, R199, R201, R30, R32: value 10k -> 47k
- R35, R83: value 1 -> 47k
- R46, R48, R89, R90: value 2.2k -> 1; device SparkFun-Resistors:0402-TIGHT -> SparkFun-Resistors:0603@1
- R49, R91: value 2.2k -> 470; device SparkFun-Resistors:0402-TIGHT -> SparkFun-Resistors:0603@1
- R85: value 470 -> 47k
- U$100, U$206: device buzzard_labels:GND3 -> buzzard_labels (1):X0
- U$101, U$207: device buzzard_labels:#MTR_RST5 -> buzzard_labels (1):Y1
- U$102, U$208: device buzzard_labels:#FSYNC7 -> buzzard_labels (1):Z2
- U$112: device buzzard_labels:#ENC_RST4 -> buzzard_labels (1):G5
- U$113: device buzzard_labels:#ENC_INT6 -> buzzard_labels (1):A4
- U$114: device buzzard_labels (1):EXT_PWR_INPUTS3 -> buzzard_labels:GND3
- U$115: device buzzard_labels (1):5V2 -> buzzard_labels:GND3
- U$116: device buzzard_labels (1):MTR1 -> buzzard_labels:GND3
- U$117: device buzzard_labels (1):SERVO0 -> buzzard_labels:#MTR_RST5
- U$118: device buzzard_labels (2):B15 -> buzzard_labels:#FSYNC7
- U$119: device buzzard_labels (2):B15 -> buzzard_labels:#ENC_RST4
- U$120: device buzzard_labels (2):ENC112 -> buzzard_labels:#ENC_INT6
- U$121, U$250: device buzzard_labels (2):ENC213 -> buzzard_labels (1):EXT_PWR_INPUTS3
- U$131: device buzzard_labels (2):A14 -> buzzard_labels (1):5V2
- U$132: device buzzard_labels (2):A14 -> buzzard_labels (1):MTR1
- U$133: device buzzard_labels (3):MTRA0 -> buzzard_labels (1):SERVO0
- U$134: device buzzard_labels (3):MTRB1 -> buzzard_labels (2):B15
- U$135: device buzzard_labels (4):10 -> buzzard_labels (2):B15
- U$136: device buzzard_labels (4):10 -> buzzard_labels (2):ENC112
- U$137: device buzzard_labels (4):21 -> buzzard_labels (2):ENC213
- U$138, U$169: device buzzard_labels (4):21 -> buzzard_labels (2):A14
- U$139: device buzzard_labels (5):00 -> buzzard_labels (2):A14
- U$140: device buzzard_labels (5):11 -> buzzard_labels (3):MTRA0
- U$141: device buzzard_labels (5):22 -> buzzard_labels (3):MTRB1
- U$142, U$173: device buzzard_labels (5):33 -> buzzard_labels (4):10
- U$143: device buzzard_labels (6):ENC_INT12 -> buzzard_labels (4):10
- U$144: device buzzard_labels (6):ENC_ADR11 -> buzzard_labels (4):21
- U$145: device buzzard_labels (6):FUSE_BP10 -> buzzard_labels (4):21
- U$146: device buzzard_labels (6):IMU_ADR9 -> buzzard_labels (5):00
- U$147: device buzzard_labels (7):MTR_ADR0 -> buzzard_labels (5):11
- U$148: device buzzard_labels (1):EXT_PWR_INPUTS3 -> buzzard_labels (5):22
- U$149: device buzzard_labels (6):5V3 -> buzzard_labels (5):33
- U$150: device buzzard_labels (6):MTR4 -> buzzard_labels (6):ENC_INT12
- U$151: device buzzard_labels (6):SERVO5 -> buzzard_labels (6):ENC_ADR11
- U$152: device buzzard_labels (6):#ENC_RST6 -> buzzard_labels (6):FUSE_BP10
- U$153: device buzzard_labels (6):#MTR_RST7 -> buzzard_labels (6):IMU_ADR9
- U$154: device buzzard_labels (6):#FSYNC8 -> buzzard_labels (7):MTR_ADR0
- U$155: device buzzard_labels:GND3 -> buzzard_labels (1):EXT_PWR_INPUTS3
- U$156: device buzzard_labels:GND3 -> buzzard_labels (6):5V3
- U$157: device buzzard_labels:GND3 -> buzzard_labels (6):#ENC_RST6
- U$158: device buzzard_labels (8):#ENC_INT0 -> buzzard_labels (6):#MTR_RST7
- U$159: device buzzard_labels (2):B15 -> buzzard_labels (6):#FSYNC8
- U$160: device buzzard_labels (2):B15 -> buzzard_labels:GND3
- U$161: device buzzard_labels (2):ENC112 -> buzzard_labels:GND3
- U$162, U$218: device buzzard_labels (2):ENC213 -> buzzard_labels:GND3
- U$163: device buzzard_labels (2):A14 -> buzzard_labels (8):#ENC_INT0
- U$164, U$515: device buzzard_labels (2):A14 -> buzzard_labels (2):B15
- U$165: device buzzard_labels (3):MTRA0 -> buzzard_labels (2):B15
- U$166: device buzzard_labels (3):MTRB1 -> buzzard_labels (2):ENC112
- U$167: device buzzard_labels (4):10 -> buzzard_labels (2):ENC213
- U$168, U$519: device buzzard_labels (4):10 -> buzzard_labels (2):A14
- U$170: device buzzard_labels (4):21 -> buzzard_labels (3):MTRA0
- U$171: device buzzard_labels (5):00 -> buzzard_labels (3):MTRB1
- U$172: device buzzard_labels (5):22 -> buzzard_labels (4):10
- U$174: device buzzard_labels (5):11 -> buzzard_labels (4):21
- U$175: device robohat:AUTOHAT-LOGO -> buzzard_labels (4):21
- U$176: device robohat:AUTOHAT-LOGO -> buzzard_labels (5):00
- U$177: value QWIIC_LOGO_5MM -> (none); device SparkFun-Aesthetics:QWIIC_5MM -> buzzard_labels (5):22
- U$178: device Qwiic RFID - IDXXLA:I_SUPER2_C-()-03 -> buzzard_labels (5):33
- U$179: device buzzard_labels (3):ISO1 -> buzzard_labels (5):11
- U$18: value QWIIC_LOGO_5MM -> (none); device SparkFun-Aesthetics:QWIIC_5MM -> autophat:1X06_2.54_SCREWTERM_PIN_REF
- U$180: device buzzard_labels (3):PI0 -> robohat:AUTOHAT-LOGO
- U$181: device buzzard_labels:STAT4 -> robohat:AUTOHAT-LOGO
- U$182: device buzzard_labels:05 -> autophat:1X06_2.54_SCREWTERM_PIN_REF
- U$183: device buzzard_labels:16 -> autophat:1X06_2.54_SCREWTERM_PIN_REF
- U$184: device buzzard_labels:27 -> buzzard_labels:SRV_5#6V1
- U$185: device buzzard_labels:38 -> buzzard_labels (1):MTR_5#9V0
- U$186, U$196: device buzzard_labels (1):X0 -> buzzard_labels:05
- U$187, U$197: device buzzard_labels (1):Y1 -> buzzard_labels:16
- U$188, U$198: device buzzard_labels (1):Z2 -> buzzard_labels:27
- U$189: device buzzard_labels (1):G5 -> buzzard_labels (3):MTR0
- U$19: device Qwiic RFID - IDXXLA:I_SUPER2_C-()-03 -> autophat:1X06_2.54_SCREWTERM_PIN_REF
- U$190: device buzzard_labels (1):A4 -> buzzard_labels (4):SRV_ADR0
- U$191: value (none) -> QWIIC_LOGO_5MM; device buzzard_labels (1):M3 -> SparkFun-Aesthetics:QWIIC_5MM
- U$192, U$287: device buzzard_labels (1):X0 -> Qwiic RFID - IDXXLA:I_SUPER2_C-()-03
- U$193, U$288: device buzzard_labels (1):Y1 -> buzzard_labels (3):ISO1
- U$194, U$289: device buzzard_labels (1):Z2 -> buzzard_labels (3):PI0
- U$195: device buzzard_labels (1):M3 -> buzzard_labels:STAT4
- U$199, U$86: device buzzard_labels (1):X0 -> buzzard_labels:38
- U$200, U$87: device buzzard_labels (1):Y1 -> buzzard_labels (1):X0
- U$201, U$88: device buzzard_labels (1):Z2 -> buzzard_labels (1):Y1
- U$202: device buzzard_labels (1):G5 -> buzzard_labels (1):Z2
- U$203: device buzzard_labels (1):A4 -> buzzard_labels (1):G5
- U$204: device buzzard_labels:GND3 -> buzzard_labels (1):A4
- U$205: device buzzard_labels:GND3 -> buzzard_labels (1):M3
- U$209: device buzzard_labels:#ENC_RST4 -> buzzard_labels (1):M3
- U$210: device buzzard_labels:#ENC_INT6 -> buzzard_labels (1):X0
- U$211: device buzzard_labels (1):EXT_PWR_INPUTS3 -> buzzard_labels (1):Y1
- U$212: device buzzard_labels (1):5V2 -> buzzard_labels (1):Z2
- U$213, U$301: device buzzard_labels (1):MTR1 -> buzzard_labels (1):X0
- U$214, U$302: device buzzard_labels (1):SERVO0 -> buzzard_labels (1):Y1
- U$215, U$303, U$392: device buzzard_labels (2):B15 -> buzzard_labels (1):Z2
- U$216: device buzzard_labels (2):B15 -> buzzard_labels (1):G5
- U$217: device buzzard_labels (2):ENC112 -> buzzard_labels (1):A4
- U$219, U$220: device buzzard_labels (2):A14 -> buzzard_labels:GND3
- U$221: device buzzard_labels (3):MTRA0 -> buzzard_labels:#MTR_RST5
- U$222: device buzzard_labels (3):MTRB1 -> buzzard_labels:#FSYNC7
- U$223: device buzzard_labels (4):10 -> buzzard_labels:#ENC_RST4
- U$224: device buzzard_labels (4):10 -> buzzard_labels:#ENC_INT6
- U$225, U$345: device buzzard_labels (4):21 -> buzzard_labels (1):EXT_PWR_INPUTS3
- U$226: device buzzard_labels (4):21 -> buzzard_labels (1):5V2
- U$227: device buzzard_labels (5):00 -> buzzard_labels (1):MTR1
- U$228: device buzzard_labels (5):11 -> buzzard_labels (1):SERVO0
- U$229, U$260: device buzzard_labels (5):22 -> buzzard_labels (2):B15
- U$230: device buzzard_labels (5):33 -> buzzard_labels (2):B15
- U$231: device buzzard_labels (6):ENC_INT12 -> buzzard_labels (2):ENC112
- U$232: device buzzard_labels (6):ENC_ADR11 -> buzzard_labels (2):ENC213
- U$233: device buzzard_labels (6):FUSE_BP10 -> buzzard_labels (2):A14
- U$234: device buzzard_labels (6):IMU_ADR9 -> buzzard_labels (2):A14
- U$235: device buzzard_labels (7):MTR_ADR0 -> buzzard_labels (3):MTRA0
- U$236: device buzzard_labels (1):EXT_PWR_INPUTS3 -> buzzard_labels (3):MTRB1
- U$237: device buzzard_labels (6):5V3 -> buzzard_labels (4):10
- U$238: device buzzard_labels (6):MTR4 -> buzzard_labels (4):10
- U$239: device buzzard_labels (6):SERVO5 -> buzzard_labels (4):21
- U$240: device buzzard_labels (6):#ENC_RST6 -> buzzard_labels (4):21
- U$241: device buzzard_labels (6):#MTR_RST7 -> buzzard_labels (5):00
- U$242: device buzzard_labels (6):#FSYNC8 -> buzzard_labels (5):11
- U$243: device buzzard_labels:GND3 -> buzzard_labels (5):22
- U$244: device buzzard_labels:GND3 -> buzzard_labels (5):33
- U$245: device buzzard_labels:GND3 -> buzzard_labels (6):ENC_INT12
- U$246: device buzzard_labels (8):#ENC_INT0 -> buzzard_labels (6):ENC_ADR11
- U$247: device buzzard_labels (2):B15 -> buzzard_labels (6):FUSE_BP10
- U$248: device buzzard_labels (2):B15 -> buzzard_labels (6):IMU_ADR9
- U$249: device buzzard_labels (2):ENC112 -> buzzard_labels (7):MTR_ADR0
- U$251: device buzzard_labels (2):A14 -> buzzard_labels (6):5V3
- U$252: device buzzard_labels (2):A14 -> buzzard_labels (6):#ENC_RST6
- U$253: device buzzard_labels (3):MTRA0 -> buzzard_labels (6):#MTR_RST7
- U$254: device buzzard_labels (3):MTRB1 -> buzzard_labels (6):#FSYNC8
- U$255, U$256: device buzzard_labels (4):10 -> buzzard_labels:GND3
- U$257, U$313, U$314: device buzzard_labels (4):21 -> buzzard_labels:GND3
- U$258: device buzzard_labels (4):21 -> buzzard_labels (8):#ENC_INT0
- U$259: device buzzard_labels (5):00 -> buzzard_labels (2):B15
- U$261: device buzzard_labels (5):33 -> buzzard_labels (2):ENC112
- U$262: device buzzard_labels (5):11 -> buzzard_labels (2):ENC213
- U$263, U$264: device robohat:AUTOHAT-LOGO -> buzzard_labels (2):A14
- U$265: value QWIIC_LOGO_5MM -> (none); device SparkFun-Aesthetics:QWIIC_5MM -> buzzard_labels (3):MTRA0
- U$266: device Qwiic RFID - IDXXLA:I_SUPER2_C-()-03 -> buzzard_labels (3):MTRB1
- U$267: device buzzard_labels (3):ISO1 -> buzzard_labels (4):10
- U$268: device buzzard_labels (3):PI0 -> buzzard_labels (4):10
- U$269: device buzzard_labels:STAT4 -> buzzard_labels (4):21
- U$270: device buzzard_labels:05 -> buzzard_labels (4):21
- U$271: device buzzard_labels:16 -> buzzard_labels (5):00
- U$272: device buzzard_labels:27 -> buzzard_labels (5):22
- U$273: device buzzard_labels:38 -> buzzard_labels (5):33
- U$274: device buzzard_labels (1):X0 -> buzzard_labels (5):11
- U$275: device buzzard_labels (1):Y1 -> robohat:AUTOHAT-LOGO
- U$276, U$370, U$465: device buzzard_labels (1):Z2 -> robohat:AUTOHAT-LOGO
- U$277: device buzzard_labels (1):G5 -> autophat:1X06_2.54_SCREWTERM_PIN_REF
- U$278, U$467: device buzzard_labels (1):A4 -> autophat:1X06_2.54_SCREWTERM_PIN_REF
- U$279: device buzzard_labels (1):M3 -> buzzard_labels:SRV_5#6V1
- U$28: value (none) -> QWIIC_LOGO_5MM; device buzzard_labels (3):ISO1 -> SparkFun-Aesthetics:QWIIC_5MM
- U$280, U$375: device buzzard_labels (1):X0 -> buzzard_labels (1):MTR_5#9V0
- U$281, U$376: device buzzard_labels (1):Y1 -> buzzard_labels:05
- U$282, U$377: device buzzard_labels (1):Z2 -> buzzard_labels:16
- U$283, U$84: device buzzard_labels (1):M3 -> buzzard_labels:27
- U$284: device buzzard_labels (1):X0 -> buzzard_labels (3):MTR0
- U$285: device buzzard_labels (1):Y1 -> buzzard_labels (4):SRV_ADR0
- U$286: value (none) -> QWIIC_LOGO_5MM; device buzzard_labels (1):Z2 -> SparkFun-Aesthetics:QWIIC_5MM
- U$290: device buzzard_labels (1):G5 -> buzzard_labels:STAT4
- U$291: device buzzard_labels (1):A4 -> buzzard_labels:05
- U$292: device buzzard_labels:GND3 -> buzzard_labels:16
- U$293: device buzzard_labels:GND3 -> buzzard_labels:27
- U$294: device buzzard_labels:GND3 -> buzzard_labels:38
- U$295: device buzzard_labels:#MTR_RST5 -> buzzard_labels (1):X0
- U$296: device buzzard_labels:#FSYNC7 -> buzzard_labels (1):Y1
- U$297: device buzzard_labels:#ENC_RST4 -> buzzard_labels (1):Z2
- U$298: device buzzard_labels:#ENC_INT6 -> buzzard_labels (1):G5
- U$299: device buzzard_labels (1):EXT_PWR_INPUTS3 -> buzzard_labels (1):A4
- U$30: device buzzard_labels (3):PI0 -> buzzard_labels:SRV_5#6V1
- U$300: device buzzard_labels (1):5V2 -> buzzard_labels (1):M3
- U$304: device buzzard_labels (2):B15 -> buzzard_labels (1):M3
- U$305: device buzzard_labels (2):ENC112 -> buzzard_labels (1):X0
- U$306: device buzzard_labels (2):ENC213 -> buzzard_labels (1):Y1
- U$307: device buzzard_labels (2):A14 -> buzzard_labels (1):Z2
- U$308, U$396: device buzzard_labels (2):A14 -> buzzard_labels (1):X0
- U$309, U$397: device buzzard_labels (3):MTRA0 -> buzzard_labels (1):Y1
- U$310, U$398: device buzzard_labels (3):MTRB1 -> buzzard_labels (1):Z2
- U$311, U$488: device buzzard_labels (4):10 -> buzzard_labels (1):G5
- U$312: device buzzard_labels (4):10 -> buzzard_labels (1):A4
- U$315: device buzzard_labels (5):00 -> buzzard_labels:GND3
- U$316: device buzzard_labels (5):11 -> buzzard_labels:#MTR_RST5
- U$317: device buzzard_labels (5):22 -> buzzard_labels:#FSYNC7
- U$318: device buzzard_labels (5):33 -> buzzard_labels:#ENC_RST4
- U$319: device buzzard_labels (6):ENC_INT12 -> buzzard_labels:#ENC_INT6
- U$320: device buzzard_labels (6):ENC_ADR11 -> buzzard_labels (1):EXT_PWR_INPUTS3
- U$321: device buzzard_labels (6):FUSE_BP10 -> buzzard_labels (1):5V2
- U$322: device buzzard_labels (6):IMU_ADR9 -> buzzard_labels (1):MTR1
- U$323: device buzzard_labels (7):MTR_ADR0 -> buzzard_labels (1):SERVO0
- U$324: device buzzard_labels (1):EXT_PWR_INPUTS3 -> buzzard_labels (2):B15
- U$325: device buzzard_labels (6):5V3 -> buzzard_labels (2):B15
- U$326: device buzzard_labels (6):MTR4 -> buzzard_labels (2):ENC112
- U$327: device buzzard_labels (6):SERVO5 -> buzzard_labels (2):ENC213
- U$328: device buzzard_labels (6):#ENC_RST6 -> buzzard_labels (2):A14
- U$329: device buzzard_labels (6):#MTR_RST7 -> buzzard_labels (2):A14
- U$330: device buzzard_labels (6):#FSYNC8 -> buzzard_labels (3):MTRA0
- U$331: device buzzard_labels:GND3 -> buzzard_labels (3):MTRB1
- U$332, U$333: device buzzard_labels:GND3 -> buzzard_labels (4):10
- U$334: device buzzard_labels (8):#ENC_INT0 -> buzzard_labels (4):21
- U$335: device buzzard_labels (2):B15 -> buzzard_labels (4):21
- U$336: device buzzard_labels (2):B15 -> buzzard_labels (5):00
- U$337: device buzzard_labels (2):ENC112 -> buzzard_labels (5):11
- U$338: device buzzard_labels (2):ENC213 -> buzzard_labels (5):22
- U$339: device buzzard_labels (2):A14 -> buzzard_labels (5):33
- U$340: device buzzard_labels (2):A14 -> buzzard_labels (6):ENC_INT12
- U$341: device buzzard_labels (3):MTRA0 -> buzzard_labels (6):ENC_ADR11
- U$342: device buzzard_labels (3):MTRB1 -> buzzard_labels (6):FUSE_BP10
- U$343: device buzzard_labels (4):10 -> buzzard_labels (6):IMU_ADR9
- U$344: device buzzard_labels (4):10 -> buzzard_labels (7):MTR_ADR0
- U$346: device buzzard_labels (4):21 -> buzzard_labels (6):5V3
- U$347: device buzzard_labels (5):00 -> buzzard_labels (6):#ENC_RST6
- U$348: device buzzard_labels (5):22 -> buzzard_labels (6):#MTR_RST7
- U$349: device buzzard_labels (5):33 -> buzzard_labels (6):#FSYNC8
- U$350: device buzzard_labels (5):11 -> buzzard_labels:GND3
- U$351, U$352: device robohat:AUTOHAT-LOGO -> buzzard_labels:GND3
- U$353: value QWIIC_LOGO_5MM -> (none); device SparkFun-Aesthetics:QWIIC_5MM -> buzzard_labels (8):#ENC_INT0
- U$354: device Qwiic RFID - IDXXLA:I_SUPER2_C-()-03 -> buzzard_labels (2):B15
- U$355: device buzzard_labels (3):ISO1 -> buzzard_labels (2):B15
- U$356: device buzzard_labels (3):PI0 -> buzzard_labels (2):ENC112
- U$357: device buzzard_labels:STAT4 -> buzzard_labels (2):ENC213
- U$358: device buzzard_labels:05 -> buzzard_labels (2):A14
- U$359: device buzzard_labels:16 -> buzzard_labels (2):A14
- U$360: device buzzard_labels:27 -> buzzard_labels (3):MTRA0
- U$361: device buzzard_labels:38 -> buzzard_labels (3):MTRB1
- U$362: device buzzard_labels (1):X0 -> buzzard_labels (4):10
- U$363, U$457: device buzzard_labels (1):Y1 -> buzzard_labels (4):10
- U$364: device buzzard_labels (1):Z2 -> buzzard_labels (4):21
- U$365: device buzzard_labels (1):G5 -> buzzard_labels (4):21
- U$366: device buzzard_labels (1):A4 -> buzzard_labels (5):00
- U$367: device buzzard_labels (1):M3 -> buzzard_labels (5):22
- U$368, U$463: device buzzard_labels (1):X0 -> buzzard_labels (5):33
- U$369, U$464: device buzzard_labels (1):Y1 -> buzzard_labels (5):11
- U$371: device buzzard_labels (1):M3 -> robohat:AUTOHAT-LOGO
- U$372: device buzzard_labels (1):X0 -> autophat:1X06_2.54_SCREWTERM_PIN_REF
- U$373: device buzzard_labels (1):Y1 -> autophat:1X06_2.54_SCREWTERM_PIN_REF
- U$374: device buzzard_labels (1):Z2 -> buzzard_labels:SRV_5#6V1
- U$378: device buzzard_labels (1):G5 -> buzzard_labels:27
- U$379: device buzzard_labels (1):A4 -> buzzard_labels (3):MTR0
- U$38: device buzzard_labels:STAT4 -> buzzard_labels (1):MTR_5#9V0
- U$380: device buzzard_labels:GND3 -> buzzard_labels (4):SRV_ADR0
- U$381: value (none) -> QWIIC_LOGO_5MM; device buzzard_labels:GND3 -> SparkFun-Aesthetics:QWIIC_5MM
- U$382: device buzzard_labels:GND3 -> Qwiic RFID - IDXXLA:I_SUPER2_C-()-03
- U$383: device buzzard_labels:#MTR_RST5 -> buzzard_labels (3):ISO1
- U$384: device buzzard_labels:#FSYNC7 -> buzzard_labels (3):PI0
- U$385: device buzzard_labels:#ENC_RST4 -> buzzard_labels:STAT4
- U$386: device buzzard_labels:#ENC_INT6 -> buzzard_labels:05
- U$387: device buzzard_labels (1):EXT_PWR_INPUTS3 -> buzzard_labels:16
- U$388: device buzzard_labels (1):5V2 -> buzzard_labels:27
- U$389: device buzzard_labels (1):MTR1 -> buzzard_labels:38
- U$390: device buzzard_labels (1):SERVO0 -> buzzard_labels (1):X0
- U$391: device buzzard_labels (2):B15 -> buzzard_labels (1):Y1
- U$393: device buzzard_labels (2):ENC112 -> buzzard_labels (1):G5
- U$394: device buzzard_labels (2):ENC213 -> buzzard_labels (1):A4
- U$395: device buzzard_labels (2):A14 -> buzzard_labels (1):M3
- U$399: device buzzard_labels (4):10 -> buzzard_labels (1):M3
- U$400: device buzzard_labels (4):10 -> buzzard_labels (1):X0
- U$401: device buzzard_labels (4):21 -> buzzard_labels (1):Y1
- U$402: device buzzard_labels (4):21 -> buzzard_labels (1):Z2
- U$403, U$491: device buzzard_labels (5):00 -> buzzard_labels (1):X0
- U$404, U$492: device buzzard_labels (5):11 -> buzzard_labels (1):Y1
- U$405, U$493: device buzzard_labels (5):22 -> buzzard_labels (1):Z2
- U$406: device buzzard_labels (5):33 -> buzzard_labels (1):G5
- U$407: device buzzard_labels (6):ENC_INT12 -> buzzard_labels (1):A4
- U$408: device buzzard_labels (6):ENC_ADR11 -> buzzard_labels:GND3
- U$409: device buzzard_labels (6):FUSE_BP10 -> buzzard_labels:GND3
- U$410: device buzzard_labels (6):IMU_ADR9 -> buzzard_labels:GND3
- U$411: device buzzard_labels (7):MTR_ADR0 -> buzzard_labels:#MTR_RST5
- U$412: device buzzard_labels (1):EXT_PWR_INPUTS3 -> buzzard_labels:#FSYNC7
- U$413: device buzzard_labels (6):5V3 -> buzzard_labels:#ENC_RST4
- U$414: device buzzard_labels (6):MTR4 -> buzzard_labels:#ENC_INT6
- U$415: device buzzard_labels (6):SERVO5 -> buzzard_labels (1):EXT_PWR_INPUTS3
- U$416: device buzzard_labels (6):#ENC_RST6 -> buzzard_labels (1):5V2
- U$417: device buzzard_labels (6):#MTR_RST7 -> buzzard_labels (1):MTR1
- U$418: device buzzard_labels (6):#FSYNC8 -> buzzard_labels (1):SERVO0
- U$419, U$420: device buzzard_labels:GND3 -> buzzard_labels (2):B15
- U$421: device buzzard_labels:GND3 -> buzzard_labels (2):ENC112
- U$422: device buzzard_labels (8):#ENC_INT0 -> buzzard_labels (2):ENC213
- U$423, U$424: device buzzard_labels (2):B15 -> buzzard_labels (2):A14
- U$425: device buzzard_labels (2):ENC112 -> buzzard_labels (3):MTRA0
- U$426: device buzzard_labels (2):ENC213 -> buzzard_labels (3):MTRB1
- U$427, U$428: device buzzard_labels (2):A14 -> buzzard_labels (4):10
- U$429: device buzzard_labels (3):MTRA0 -> buzzard_labels (4):21
- U$430: device buzzard_labels (3):MTRB1 -> buzzard_labels (4):21
- U$431: device buzzard_labels (4):10 -> buzzard_labels (5):00
- U$432: device buzzard_labels (4):10 -> buzzard_labels (5):11
- U$433: device buzzard_labels (4):21 -> buzzard_labels (5):22
- U$434: device buzzard_labels (4):21 -> buzzard_labels (5):33
- U$435: device buzzard_labels (5):00 -> buzzard_labels (6):ENC_INT12
- U$436: device buzzard_labels (5):22 -> buzzard_labels (6):ENC_ADR11
- U$437: device buzzard_labels (5):33 -> buzzard_labels (6):FUSE_BP10
- U$438: device buzzard_labels (5):11 -> buzzard_labels (6):IMU_ADR9
- U$439: device robohat:AUTOHAT-LOGO -> buzzard_labels (7):MTR_ADR0
- U$440: device robohat:AUTOHAT-LOGO -> buzzard_labels (1):EXT_PWR_INPUTS3
- U$441: value QWIIC_LOGO_5MM -> (none); device SparkFun-Aesthetics:QWIIC_5MM -> buzzard_labels (6):5V3
- U$442: device Qwiic RFID - IDXXLA:I_SUPER2_C-()-03 -> buzzard_labels (6):#ENC_RST6
- U$443: device buzzard_labels (3):ISO1 -> buzzard_labels (6):#MTR_RST7
- U$444: device buzzard_labels (3):PI0 -> buzzard_labels (6):#FSYNC8
- U$445: device buzzard_labels:STAT4 -> buzzard_labels:GND3
- U$446: device buzzard_labels:05 -> buzzard_labels:GND3
- U$447: device buzzard_labels:16 -> buzzard_labels:GND3
- U$448: device buzzard_labels:27 -> buzzard_labels (8):#ENC_INT0
- U$449: device buzzard_labels:38 -> buzzard_labels (2):B15
- U$450: device buzzard_labels (1):X0 -> buzzard_labels (2):B15
- U$451: device buzzard_labels (1):Y1 -> buzzard_labels (2):ENC112
- U$452: device buzzard_labels (1):Z2 -> buzzard_labels (2):ENC213
- U$453: device buzzard_labels (1):G5 -> buzzard_labels (2):A14
- U$454: device buzzard_labels (1):A4 -> buzzard_labels (2):A14
- U$455: device buzzard_labels (1):M3 -> buzzard_labels (3):MTRA0
- U$456: device buzzard_labels (1):X0 -> buzzard_labels (3):MTRB1
- U$458: device buzzard_labels (1):Z2 -> buzzard_labels (4):10
- U$459: device buzzard_labels (1):M3 -> buzzard_labels (4):21
- U$46: device buzzard_labels:38 -> buzzard_labels (3):MTR0
- U$460: device buzzard_labels (1):X0 -> buzzard_labels (4):21
- U$461: device buzzard_labels (1):Y1 -> buzzard_labels (5):00
- U$462: device buzzard_labels (1):Z2 -> buzzard_labels (5):22
- U$466: device buzzard_labels (1):G5 -> robohat:AUTOHAT-LOGO
- U$468: device buzzard_labels:GND3 -> autophat:1X06_2.54_SCREWTERM_PIN_REF
- U$469: device buzzard_labels:GND3 -> buzzard_labels:SRV_5#6V1
- U$47: device buzzard_labels (1):X0 -> buzzard_labels (4):SRV_ADR0
- U$470: device buzzard_labels:GND3 -> buzzard_labels (1):MTR_5#9V0
- U$471: device buzzard_labels:#MTR_RST5 -> buzzard_labels:05
- U$472: device buzzard_labels:#FSYNC7 -> buzzard_labels:16
- U$473: device buzzard_labels:#ENC_RST4 -> buzzard_labels:27
- U$474: device buzzard_labels:#ENC_INT6 -> buzzard_labels (3):MTR0
- U$475: device buzzard_labels (1):EXT_PWR_INPUTS3 -> buzzard_labels (4):SRV_ADR0
- U$476: value (none) -> QWIIC_LOGO_5MM; device buzzard_labels (1):5V2 -> SparkFun-Aesthetics:QWIIC_5MM
- U$477: device buzzard_labels (1):MTR1 -> Qwiic RFID - IDXXLA:I_SUPER2_C-()-03
- U$478: device buzzard_labels (1):SERVO0 -> buzzard_labels (3):ISO1
- U$479: device buzzard_labels (2):B15 -> buzzard_labels (3):PI0
- U$480: device buzzard_labels (2):B15 -> buzzard_labels:STAT4
- U$481: device buzzard_labels (2):ENC112 -> buzzard_labels:05
- U$482: device buzzard_labels (2):ENC213 -> buzzard_labels:16
- U$483: device buzzard_labels (2):A14 -> buzzard_labels:27
- U$484: device buzzard_labels (2):A14 -> buzzard_labels:38
- U$485: device buzzard_labels (3):MTRA0 -> buzzard_labels (1):X0
- U$486: device buzzard_labels (3):MTRB1 -> buzzard_labels (1):Y1
- U$487: device buzzard_labels (4):10 -> buzzard_labels (1):Z2
- U$489: device buzzard_labels (4):21 -> buzzard_labels (1):A4
- U$490: device buzzard_labels (4):21 -> buzzard_labels (1):M3
- U$494: device buzzard_labels (5):33 -> buzzard_labels (1):M3
- U$495: device buzzard_labels (6):ENC_INT12 -> buzzard_labels (1):X0
- U$496: device buzzard_labels (6):ENC_ADR11 -> buzzard_labels (1):Y1
- U$497: device buzzard_labels (6):FUSE_BP10 -> buzzard_labels (1):Z2
- U$498: device buzzard_labels (6):IMU_ADR9 -> buzzard_labels (1):X0
- U$499: device buzzard_labels (7):MTR_ADR0 -> buzzard_labels (1):Y1
- U$500: device buzzard_labels (1):EXT_PWR_INPUTS3 -> buzzard_labels (1):Z2
- U$501: device buzzard_labels (6):5V3 -> buzzard_labels (1):G5
- U$502: device buzzard_labels (6):MTR4 -> buzzard_labels (1):A4
- U$503: device buzzard_labels (6):SERVO5 -> buzzard_labels:GND3
- U$504: device buzzard_labels (6):#ENC_RST6 -> buzzard_labels:GND3
- U$505: device buzzard_labels (6):#MTR_RST7 -> buzzard_labels:GND3
- U$506: device buzzard_labels (6):#FSYNC8 -> buzzard_labels:#MTR_RST5
- U$507: device buzzard_labels:GND3 -> buzzard_labels:#FSYNC7
- U$508: device buzzard_labels:GND3 -> buzzard_labels:#ENC_RST4
- U$509: device buzzard_labels:GND3 -> buzzard_labels:#ENC_INT6
- U$510: device buzzard_labels (8):#ENC_INT0 -> buzzard_labels (1):EXT_PWR_INPUTS3
- U$511: device buzzard_labels (2):B15 -> buzzard_labels (1):5V2
- U$512: device buzzard_labels (2):B15 -> buzzard_labels (1):MTR1
- U$513: device buzzard_labels (2):ENC112 -> buzzard_labels (1):SERVO0
- U$514: device buzzard_labels (2):ENC213 -> buzzard_labels (2):B15
- U$516: device buzzard_labels (2):A14 -> buzzard_labels (2):ENC112
- U$517: device buzzard_labels (3):MTRA0 -> buzzard_labels (2):ENC213
- U$518: device buzzard_labels (3):MTRB1 -> buzzard_labels (2):A14
- U$520: device buzzard_labels (4):10 -> buzzard_labels (3):MTRA0
- U$521: device buzzard_labels (4):21 -> buzzard_labels (3):MTRB1
- U$522: device buzzard_labels (4):21 -> buzzard_labels (4):10
- U$523: device buzzard_labels (5):00 -> buzzard_labels (4):10
- U$524: device buzzard_labels (5):22 -> buzzard_labels (4):21
- U$525: device buzzard_labels (5):33 -> buzzard_labels (4):21
- U$526: device buzzard_labels (5):11 -> buzzard_labels (5):00
- U$527: device robohat:AUTOHAT-LOGO -> buzzard_labels (5):11
- U$528: device robohat:AUTOHAT-LOGO -> buzzard_labels (5):22
- U$54: device buzzard_labels (6):MTR4 -> Qwiic RFID - IDXXLA:I_SUPER2_C-()-03
- U$55: device buzzard_labels (6):SERVO5 -> buzzard_labels (3):ISO1
- U$63: device buzzard_labels (1):Y1 -> buzzard_labels (3):PI0
- U$64: device buzzard_labels (1):Z2 -> buzzard_labels:STAT4
- U$71: device buzzard_labels (1):G5 -> buzzard_labels:05
- U$72: device buzzard_labels (1):A4 -> buzzard_labels:16
- U$89: device buzzard_labels (1):M3 -> buzzard_labels (1):Z2
- U$90: device buzzard_labels (1):X0 -> buzzard_labels (1):G5
- U$91: device buzzard_labels (1):Y1 -> buzzard_labels (1):A4
- U$92: device buzzard_labels (1):Z2 -> buzzard_labels (1):M3
- U$96: device buzzard_labels (1):G5 -> buzzard_labels (1):M3
- U$97: device buzzard_labels (1):A4 -> buzzard_labels (1):X0
- U$98: device buzzard_labels:GND3 -> buzzard_labels (1):Y1
- U$99: device buzzard_labels:GND3 -> buzzard_labels (1):Z2
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Connections:
- new net ADD_A0: JP1.2, R18.1, U1.1
- new net ADD_A1: JP5.2, R17.1, U1.2
- new net ADD_A10: JP46.2, R151.1, U19.1
- new net ADD_A11: JP48.2, R152.1, U19.3
- new net ADD_A12: JP59.2, R188.1, U25.2
- new net ADD_A13: JP58.2, R189.1, U25.1
- new net ADD_A14: JP60.2, R190.1, U25.3
- new net ADD_A15: JP71.2, R226.1, U31.2
- new net ADD_A16: JP70.2, R227.1, U31.1
- new net ADD_A17: JP72.2, R228.1, U31.3
- new net ADD_A2: JP6.2, R19.1, U1.3
- new net ADD_A3: JP23.2, R74.1, U2.2
- new net ADD_A4: JP22.2, R75.1, U2.1
- new net ADD_A5: JP24.2, R76.1, U2.3
- new net ADD_A6: JP35.2, R112.1, U13.2
- new net ADD_A7: JP34.2, R113.1, U13.1
- new net ADD_A8: JP36.2, R114.1, U13.3
- new net ADD_A9: JP47.2, R150.1, U19.2
- net !ENC_INT1: now also R61.1; no longer R58.1
- net !ENC_INT2: now also R99.1; no longer R93.1
- net !ENC_INT3: now also R137.1; no longer R128.1
- net !ENC_INT4: now also R175.1; no longer R163.1
- net !ENC_INT5: now also R213.1; no longer R198.1
- net !ENC_RST1: now also R60.1; no longer R57.1
- net !ENC_RST2: now also R98.1; no longer R92.1
- net !ENC_RST3: now also R136.1; no longer R127.1
- net !ENC_RST4: now also R174.1; no longer R162.1
- net !ENC_RST5: now also R212.1; no longer R197.1
- net !FSYNC_1.8V1: now also R52.1; no longer R49.1
- net !FSYNC_1.8V2: now also R94.1; no longer R88.1
- net !FSYNC_1.8V3: now also R132.1; no longer R123.1
- net !FSYNC_1.8V4: now also R170.1; no longer R158.1
- net !FSYNC_1.8V5: now also R208.1; no longer R193.1
- net !FSYNC_3.3V1: now also R57.1; no longer R50.1
- net !FSYNC_3.3V2: now also R95.1; no longer R89.1
- net !FSYNC_3.3V3: now also R133.1; no longer R124.1
- net !FSYNC_3.3V4: now also R171.1; no longer R159.1
- net !FSYNC_3.3V5: now also R209.1; no longer R194.1
- net 1.8V1: now also R50.2, R52.2, R58.2, R73.2; no longer R46.2, R48.2, R49.2, R70.2
- net 1.8V2: now also R111.2, R92.2, R93.2, R94.2, R96.2; no longer R105.2, R86.2, R87.2, R88.2, R90.2
- net 1.8V3: now also R130.2, R131.2, R132.2, R134.2, R149.2; no longer R121.2, R122.2, R123.2, R125.2, R140.2
- net 1.8V4: now also R168.2, R169.2, R170.2, R172.2, R187.2; no longer R156.2, R157.2, R158.2, R160.2, R175.2
- net 1.8V5: now also R206.2, R207.2, R208.2, R225.2; no longer R191.2, R192.2, R193.2, R195.2
- net 3.3V1: now also JP8.2, R46.2, R48.2, R60.2, R62.2, R64.2, R66.2, R68.1, R71.2, R72.2; no longer JP5.2, R34.2, R35.2, R50.2, R52.2, R61.2, R63.2, R65.1, R68.2, R69.2
- net 3.3V2: now also JP26.2, R100.2, R102.2, R106.1, R109.2, R110.2, R90.2, R95.2, R97.2; no longer JP20.2, R100.1, R103.2, R83.2, R84.2, R91.2, R92.2, R94.2, R96.2
- net 3.3V3: now also JP38.2, R128.2, R135.2, R136.2, R140.2, R142.2, R144.1, R147.2, R148.2; no longer JP29.2, R118.2, R119.2, R124.2, R126.2, R129.2, R131.2, R135.1, R139.2
- net 3.3V4: now also JP50.2, R165.2, R171.2, R176.2, R178.2, R180.2, R182.1, R185.2, R186.2; no longer JP38.2, R153.2, R154.2, R159.2, R161.2, R162.2, R164.2, R168.2, R170.1
- net 3.3V5: now also JP62.2, R204.2, R211.2, R212.2, R214.2, R216.2, R218.2, R220.1, R223.2, R224.2; no longer JP47.2, R188.2, R189.2, R194.2, R196.2, R197.2, R199.2, R201.2, R205.1, R208.2
- net 5V: now also R17.2, R18.2, R19.2
- net 5V1: now also JP7.2, R20.2, R21.2, R74.2, R75.2, R76.2; no longer JP1.2, R17.2, R18.2
- net 5V2: now also JP25.2, R112.2, R113.2, R114.2, R77.2, R78.2; no longer JP19.2, R71.2, R72.2
- net 5V3: now also JP37.2, R115.2, R116.2, R150.2, R151.2, R152.2; no longer JP28.2, R106.2, R107.2
- net 5V4: now also JP49.2, R153.2, R154.2, R188.2, R189.2, R190.2; no longer JP37.2, R141.2, R142.2
- net 5V5: now also JP61.2, R191.2, R192.2, R226.2, R227.2, R228.2; no longer JP46.2, R176.2, R177.2
- net AD0/SDO1: now also JP20.2, R73.1; no longer JP17.2, R70.1
- net AD0/SDO2: now also JP32.2, R111.1; no longer JP26.2, R105.1
- net AD0/SDO3: now also JP44.2, R149.1; no longer JP35.2, R140.1
- net AD0/SDO4: now also JP56.2, R187.1; no longer JP44.2, R175.1
- net AD0/SDO5: now also JP68.2, R225.1; no longer JP53.2, R210.1
- net ADR1: now also JP21.2; no longer JP18.2
- net ADR2: now also JP33.2; no longer JP27.2
- net ADR3: now also JP45.2; no longer JP36.2
- net ADR4: now also JP57.2; no longer JP45.2
- net ADR5: now also JP69.2; no longer JP54.2
- net CC10: now also R158.2; no longer R146.2
- net CC11: now also R195.2; no longer R180.2
- net CC12: now also R196.2; no longer R181.2
- net CC3: now also R28.2; no longer R21.2
- net CC4: now also R29.2; no longer R23.2
- net CC5: now also R81.2; no longer R75.2
- net CC6: now also R82.2; no longer R76.2
- net CC7: now also R119.2; no longer R110.2
- net CC8: now also R120.2; no longer R111.2
- net CC9: now also R157.2; no longer R145.2
- net CONFIG_OUT1: now also R70.2; no longer R67.2
- net CONFIG_OUT2: now also R108.2; no longer R102.2
- net CONFIG_OUT3: now also R146.2; no longer R137.2
- net CONFIG_OUT4: now also R184.2; no longer R172.2
- net CONFIG_OUT5: now also R222.2; no longer R207.2
- net ENC1A_FILTERED1: now also R63.2; no longer R60.2
- net ENC1A_FILTERED2: now also R101.2; no longer R95.2
- net ENC1A_FILTERED3: now also R139.2; no longer R130.2
- net ENC1A_FILTERED4: now also R177.2; no longer R165.2
- net ENC1A_FILTERED5: now also R215.2; no longer R200.2
- net ENC1A_RAW1: now also R62.1, R63.1; no longer R59.1, R60.1
- net ENC1A_RAW2: now also R100.1, R101.1; no longer R94.1, R95.1
- net ENC1A_RAW3: now also R138.1, R139.1; no longer R129.1, R130.1
- net ENC1A_RAW4: now also R176.1, R177.1; no longer R164.1, R165.1
- net ENC1A_RAW5: now also R214.1, R215.1; no longer R199.1, R200.1
- net ENC1B_FILTERED1: now also R65.1; no longer R62.1
- net ENC1B_FILTERED2: now also R103.1; no longer R97.1
- net ENC1B_FILTERED3: now also R141.1; no longer R132.1
- net ENC1B_FILTERED4: now also R179.1; no longer R167.1
- net ENC1B_FILTERED5: now also R217.1; no longer R202.1
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Routing:
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Other:
- board size 226.4 x 136.6 mm -> 223.9 x 133.9 mm
- board text added: "v12"
- board text removed: "v11"
